Commit message: Refactor UR3e robot description and improve LLM planner API integration
- Updated the URDF Xacro file to adjust the positioning of the Robotiq gripper and coupler joints for better alignment.
- Enhanced the launch file for the UR3e LLM control to include a skill executor node and improved argument handling for starting the interactive CLI.
- Refactored the LLMPlanner class to load the OpenRouter API key from environment variables or a .env file, improving security and flexibility.
- Added error handling for API requests and improved JSON parsing from the AI response.

File: src/moveit2_ur3e/ur3e_robot_description/urdf/ur3e/robot.urdf.xacro (robot description, xacro)
@@ -24,10 +24,12 @@
     </link>
     <joint name="robotiq_coupler_joint" type="fixed">
-      <origin xyz="0 0 0.004" rpy="0 0 ${-pi/2.0}" />
+      <!-- coupler is 14 mm thick; place its lower face at the tool0 flange -->
+      <origin xyz="0 0 0.007" rpy="0 0 ${-pi/2.0}" />
       <parent link="tool0"/>
       <child link="robotiq_coupler"/>
     </joint>
     <joint name="ur3e_robotiq_2f_140_joint" type="fixed">
-      <origin xyz="0 0 0.004" rpy="0 0 ${-pi/2.0}" />
+      <!-- mount the gripper from the upper face of the coupler -->
+      <origin xyz="0 0 0.007" rpy="0 0 ${-pi/2.0}" />
       <parent link="robotiq_coupler"/>
       <child link="robotiq_arg2f_base_link"/>
